File: hardware/RPi-UNO-HAT_v11.brd (EAGLE design)
At the start: 65 x 56 mm, 61 parts, among them IC1 24LC-I/OT, IC2 ATMEGA328-AU, IC3 LDO-TS9011-3V3, Q1 16MHz, T1 BSS138PS, T2 BSS138PS, T3 BSS138PS, X1 PASSER-07, X2 PASSER-07, X3 PASSER-07

Commit message: updated layout and schematics
Routing:
- net D0_RX: track 66.2 -> 77.7 mm
Other:
- board text added: "Rev 1.1"
- board text removed: "Rev 1.0"
